File: Guess.kicad_sch (KiCad schematic)
At the start: 8 parts

Commit message: Added FSM, Button, 555 timer, changed shift registers
Parts:
- renumbered R21 to R29, R22 to R30, R23 to R31, R24 to R32, R25 to R33, R26 to R34, R27 to R35, R28 to R36
Other:
- title: (none) -> Guess Input Voltage Dividers
Changed lines of the file:
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@@
 	(generator_version "9.0")
 	(paper "A5")
+	(title_block
+		(title "Guess Input Voltage Dividers")
+		(date "2026-03-14")
+	)
 	(junction
 		(at 40.64 62.23)
@@
 		(dnp no)
 		(fields_autoplaced yes)
-		(property "Reference" "R25"
+		(property "Reference" "R33"
 			(at 93.98 55.8799 0)
 			(effects
@@
 			(project "ECE145Mastermind"
 				(path "/8c64fe8a-5d6b-41bc-b3a3-9bda7b2e0f2c/9b9c62dc-9f79-4269-b727-e91a3c4aae61"
-					(reference "R25")
+					(reference "R33")
 					(unit 1)
 				)
@@
 		(dnp no)
 		(fields_autoplaced yes)
-		(property "Reference" "#PWR019"
+		(property "Reference" "#PWR062"
 			(at 91.44 77.47 0)
 			(effects
@@
 			(project "ECE145Mastermind"
 				(path "/8c64fe8a-5d6b-41bc-b3a3-9bda7b2e0f2c/9b9c62dc-9f79-4269-b727-e91a3c4aae61"
-					(reference "#PWR019")
+					(reference "#PWR062")
 					(unit 1)
 				)
@@
 		(dnp no)
 		(fields_autoplaced yes)
-		(property "Reference" "R26"
+		(property "Reference" "R34"
 			(at 93.98 66.0399 0)
 			(effects
@@
 			(project "ECE145Mastermind"
 				(path "/8c64fe8a-5d6b-41bc-b3a3-9bda7b2e0f2c/9b9c62dc-9f79-4269-b727-e91a3c4aae61"
-					(reference "R26")
+					(reference "R34")
 					(unit 1)
 				)
@@
 		(dnp no)
 		(fields_autoplaced yes)
-		(property "Reference" "#PWR014"
+		(property "Reference" "#PWR060"
 			(at 66.04 77.47 0)
 			(effects
@@
 			(project "ECE145Mastermind"
 				(path "/8c64fe8a-5d6b-41bc-b3a3-9bda7b2e0f2c/9b9c62dc-9f79-4269-b727-e91a3c4aae61"
-					(reference "#PWR014")
+					(reference "#PWR060")
 					(unit 1)
 				)
@@
 		(dnp no)
 		(fields_autoplaced yes)
-		(property "Reference" "#PWR016"
+		(property "Reference" "#PWR058"
 			(at 40.64 77.47 0)
 			(effects
@@
 			(project ""
 				(path "/8c64fe8a-5d6b-41bc-b3a3-9bda7b2e0f2c/9b9c62dc-9f79-4269-b727-e91a3c4aae61"
-					(reference "#PWR016")
+					(reference "#PWR058")
 					(unit 1)
 				)
@@
 		(dnp no)
 		(fields_autoplaced yes)
-		(property "Reference" "#PWR022"
+		(property "Reference" "#PWR064"
 			(at 116.84 77.47 0)
 			(effects
@@
 			(project "ECE145Mastermind"
 				(path "/8c64fe8a-5d6b-41bc-b3a3-9bda7b2e0f2c/9b9c62dc-9f79-4269-b727-e91a3c4aae61"
-					(reference "#PWR022")
-					(unit 1)
-				)
-			)
-		)
-	)
-	(symbol
-		(lib_id "power:+9V")
+					(reference "#PWR064")
+					(unit 1)
+				)
+			)
+		)
+	)
+	(symbol
+		(lib_id "power:+5V")
 		(at 116.84 50.8 0)
 		(unit 1)
@@
 		(dnp no)
 		(fields_autoplaced yes)
-		(property "Reference" "#PWR021"
-			(at 116.84 54.61 0)
+		(property "Reference" "#PWR063"
+			(at 116.84 43.18 0)
 			(effects
 				(font
@@
 			)
 		)
-		(property "Description" "Power symbol creates a global label with name \"+9V\""
+		(property "Description" "Power symbol creates a global label with name \"+5V\""
 			(at 116.84 50.8 0)
 			(effects
@@
 			(project ""
 				(path "/8c64fe8a-5d6b-41bc-b3a3-9bda7b2e0f2c/9b9c62dc-9f79-4269-b727-e91a3c4aae61"
-					(reference "#PWR021")
+					(reference "#PWR063")
 					(unit 1)
 				)
@@
 		(dnp no)
 		(fields_autoplaced yes)
-		(property "Reference" "R28"
+		(property "Reference" "R36"
 			(at 119.38 66.0399 0)
 			(effects
@@
 			(project "ECE145Mastermind"
 				(path "/8c64fe8a-5d6b-41bc-b3a3-9bda7b2e0f2c/9b9c62dc-9f79-4269-b727-e91a3c4aae61"
-					(reference "R28")
+					(reference "R36")
 					(unit 1)
 				)
@@
 		(dnp no)
 		(fields_autoplaced yes)
-		(property "Reference" "R22"
+		(property "Reference" "R30"
 			(at 43.18 66.0399 0)
 			(effects
@@
 			(project "ECE145Mastermind"
 				(path "/8c64fe8a-5d6b-41bc-b3a3-9bda7b2e0f2c/9b9c62dc-9f79-4269-b727-e91a3c4aae61"
-					(reference "R22")
+					(reference "R30")
 					(unit 1)
 				)
@@
 		(dnp no)
 		(fields_autoplaced yes)
-		(property "Reference" "R27"
+		(property "Reference" "R35"
 			(at 119.38 55.8799 0)
 			(effects
@@
 			(project "ECE145Mastermind"
 				(path "/8c64fe8a-5d6b-41bc-b3a3-9bda7b2e0f2c/9b9c62dc-9f79-4269-b727-e91a3c4aae61"
-					(reference "R27")
+					(reference "R35")
 					(unit 1)
 				)
@@
 		(dnp no)
 		(fields_autoplaced yes)
-		(property "Reference" "R21"
+		(property "Reference" "R29"
 			(at 43.18 55.8799 0)
 			(effects
@@
 			(project "ECE145Mastermind"
 				(path "/8c64fe8a-5d6b-41bc-b3a3-9bda7b2e0f2c/9b9c62dc-9f79-4269-b727-e91a3c4aae61"
-					(reference "R21")
-					(unit 1)
-				)
-			)
-		)
-	)
-	(symbol
-		(lib_id "power:+9V")
+					(reference "R29")
+					(unit 1)
+				)
+			)
+		)
+	)
+	(symbol
+		(lib_id "power:+5V")
 		(at 66.04 50.8 0)
 		(unit 1)
@@
 		(dnp no)
 		(fields_autoplaced yes)
-		(property "Reference" "#PWR013"
-			(at 66.04 54.61 0)
+		(property "Reference" "#PWR059"
+			(at 66.04 43.18 0)
 			(effects
 				(font
@@
 			)
 		)
-		(property "Description" "Power symbol creates a global label with name \"+9V\""
+		(property "Description" "Power symbol creates a global label with name \"+5V\""
 			(at 66.04 50.8 0)
 			(effects
@@
 			(project ""
 				(path "/8c64fe8a-5d6b-41bc-b3a3-9bda7b2e0f2c/9b9c62dc-9f79-4269-b727-e91a3c4aae61"
-					(reference "#PWR013")
+					(reference "#PWR059")
 					(unit 1)
 				)
@@
 		(dnp no)
 		(fields_autoplaced yes)
-		(property "Reference" "R24"
+		(property "Reference" "R32"
 			(at 68.58 66.0399 0)
 			(effects
@@
 			(project "ECE145Mastermind"
 				(path "/8c64fe8a-5d6b-41bc-b3a3-9bda7b2e0f2c/9b9c62dc-9f79-4269-b727-e91a3c4aae61"
-					(reference "R24")
+					(reference "R32")
 					(unit 1)
 				)
@@
 		(dnp no)
 		(fields_autoplaced yes)
-		(property "Reference" "R23"
+		(property "Reference" "R31"
 			(at 68.58 55.8799 0)
 			(effects
@@
 			(project "ECE145Mastermind"
 				(path "/8c64fe8a-5d6b-41bc-b3a3-9bda7b2e0f2c/9b9c62dc-9f79-4269-b727-e91a3c4aae61"
-					(reference "R23")
-					(unit 1)
-				)
-			)
-		)
-	)
-	(symbol
-		(lib_id "power:+9V")
+					(reference "R31")
+					(unit 1)
+				)
+			)
+		)
+	)
+	(symbol
+		(lib_id "power:+5V")
 		(at 40.64 50.8 0)
 		(unit 1)
@@
 		(dnp no)
 		(fields_autoplaced yes)
-		(property "Reference" "#PWR011"
-			(at 40.64 54.61 0)
+		(property "Reference" "#PWR057"
+			(at 40.64 43.18 0)
 			(effects
 				(font
@@
 			)
 		)
-		(property "Description" "Power symbol creates a global label with name \"+9V\""
+		(property "Description" "Power symbol creates a global label with name \"+5V\""
 			(at 40.64 50.8 0)
 			(effects
@@
 			(project ""
 				(path "/8c64fe8a-5d6b-41bc-b3a3-9bda7b2e0f2c/9b9c62dc-9f79-4269-b727-e91a3c4aae61"
-					(reference "#PWR011")
-					(unit 1)
-				)
-			)
-		)
-	)
-	(symbol
-		(lib_id "power:+9V")
+					(reference "#PWR057")
+					(unit 1)
+				)
+			)
+		)
+	)
+	(symbol
+		(lib_id "power:+5V")
 		(at 91.44 50.8 0)
 		(unit 1)
@@
 		(dnp no)
 		(fields_autoplaced yes)
-		(property "Reference" "#PWR018"
-			(at 91.44 54.61 0)
+		(property "Reference" "#PWR061"
+			(at 91.44 43.18 0)
 			(effects
 				(font
@@
 			)
 		)
-		(property "Description" "Power symbol creates a global label with name \"+9V\""
+		(property "Description" "Power symbol creates a global label with name \"+5V\""
 			(at 91.44 50.8 0)
 			(effects
@@
 			(project ""
 				(path "/8c64fe8a-5d6b-41bc-b3a3-9bda7b2e0f2c/9b9c62dc-9f79-4269-b727-e91a3c4aae61"
-					(reference "#PWR018")
-					(unit 1)
-				)
+					(reference "#PWR061")
+					(unit 1)
+				)

Commit message: Started PCB Work
Parts:
- removed R32, R34, R36: ~, symbol Device:R
- removed R33, R35: 10k, symbol Device:R
- added J14, J15, J16, J17, J6, J7, J8, J9: Conn_01x01_Socket, Connector_PinSocket_1.27mm:PinSocket_1x01_P1.27mm_Vertical, symbol Connector:Conn_01x01_Socket
- added R28: 10k, Resistor_SMD:R_0805_2012Metric_Pad1.20x1.40mm_HandSolder, symbol Device:R
- R29, R31: footprint (none) -> Resistor_SMD:R_0805_2012Metric_Pad1.20x1.40mm_HandSolder
- R30: value ~ -> 10k; footprint (none) -> Resistor_SMD:R_0805_2012Metric_Pad1.20x1.40mm_HandSolder
Connections:
- net +5V: now also R30.1, R28.1
- net G1: now also J6.1 (Pin_1), R28.2; no longer R29.2, R30.1
- net G2: now also R29.2, J8.1 (Pin_1); no longer R31.2
- net G3: now also R30.2, J14.1 (Pin_1)
- net G4: now also R31.2, J16.1 (Pin_1)
- net GND: now also J15.1 (Pin_1), J17.1 (Pin_1), J7.1 (Pin_1), J9.1 (Pin_1); no longer R30.2

Commit message: routed
Parts:
- renumbered J6 to J10, J7 to J11, J8 to J12, J9 to J13, R28 to R29, R29 to R30, R30 to R31, R31 to R32
Changed lines of the file:
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@@
 		(dnp no)
 		(fields_autoplaced yes)
-		(property "Reference" "R29"
+		(property "Reference" "R30"
 			(at 62.23 55.8799 0)
 			(effects
@@
 			(project "ECE145Mastermind"
 				(path "/8c64fe8a-5d6b-41bc-b3a3-9bda7b2e0f2c/9b9c62dc-9f79-4269-b727-e91a3c4aae61"
-					(reference "R29")
+					(reference "R30")
 					(unit 1)
 				)
@@
 		(dnp no)
 		(fields_autoplaced yes)
-		(property "Reference" "#PWR0108"
+		(property "Reference" "#PWR0109"
 			(at 85.09 43.18 0)
 			(effects
@@
 			(project "ECE145Mastermind"
 				(path "/8c64fe8a-5d6b-41bc-b3a3-9bda7b2e0f2c/9b9c62dc-9f79-4269-b727-e91a3c4aae61"
-					(reference "#PWR0108")
+					(reference "#PWR0109")
 					(unit 1)
 				)
@@
 		(dnp no)
 		(fields_autoplaced yes)
-		(property "Reference" "R30"
+		(property "Reference" "R31"
 			(at 74.93 55.8799 0)
 			(effects
@@
 			(project "ECE145Mastermind"
 				(path "/8c64fe8a-5d6b-41bc-b3a3-9bda7b2e0f2c/9b9c62dc-9f79-4269-b727-e91a3c4aae61"
-					(reference "R30")
+					(reference "R31")
 					(unit 1)
 				)
@@
 		(dnp no)
 		(fields_autoplaced yes)
-		(property "Reference" "#PWR0102"
+		(property "Reference" "#PWR0103"
 			(at 46.99 43.18 0)
 			(effects
@@
 			(project "ECE145Mastermind"
 				(path "/8c64fe8a-5d6b-41bc-b3a3-9bda7b2e0f2c/9b9c62dc-9f79-4269-b727-e91a3c4aae61"
-					(reference "#PWR0102")
+					(reference "#PWR0103")
 					(unit 1)
 				)
@@
 		(dnp no)
 		(fields_autoplaced yes)
-		(property "Reference" "R31"
+		(property "Reference" "R32"
 			(at 87.63 55.8799 0)
 			(effects
@@
 			(project "ECE145Mastermind"
 				(path "/8c64fe8a-5d6b-41bc-b3a3-9bda7b2e0f2c/9b9c62dc-9f79-4269-b727-e91a3c4aae61"
-					(reference "R31")
+					(reference "R32")
 					(unit 1)
 				)
@@
 		(dnp no)
 		(fields_autoplaced yes)
-		(property "Reference" "J9"
+		(property "Reference" "J13"
 			(at 55.245 59.69 0)
 			(effects
@@
 			(project "ECE145Mastermind"
 				(path "/8c64fe8a-5d6b-41bc-b3a3-9bda7b2e0f2c/9b9c62dc-9f79-4269-b727-e91a3c4aae61"
-					(reference "J9")
+					(reference "J13")
 					(unit 1)
 				)
@@
 		(dnp no)
 		(fields_autoplaced yes)
-		(property "Reference" "#PWR0103"
+		(property "Reference" "#PWR0104"
 			(at 46.99 71.12 0)
 			(effects
@@
 			(project "ECE145Mastermind"
 				(path "/8c64fe8a-5d6b-41bc-b3a3-9bda7b2e0f2c/9b9c62dc-9f79-4269-b727-e91a3c4aae61"
-					(reference "#PWR0103")
+					(reference "#PWR0104")
 					(unit 1)
 				)
@@
 		(dnp no)
 		(fields_autoplaced yes)
-		(property "Reference" "J7"
+		(property "Reference" "J11"
 			(at 42.545 59.69 0)
 			(effects
@@
 			(project "ECE145Mastermind"
 				(path "/8c64fe8a-5d6b-41bc-b3a3-9bda7b2e0f2c/9b9c62dc-9f79-4269-b727-e91a3c4aae61"
-					(reference "J7")
+					(reference "J11")
 					(unit 1)
 				)
@@
 		(dnp no)
 		(fields_autoplaced yes)
-		(property "Reference" "#PWR0104"
+		(property "Reference" "#PWR0105"
 			(at 59.69 43.18 0)
 			(effects
@@
 			(project "ECE145Mastermind"
 				(path "/8c64fe8a-5d6b-41bc-b3a3-9bda7b2e0f2c/9b9c62dc-9f79-4269-b727-e91a3c4aae61"
-					(reference "#PWR0104")
+					(reference "#PWR0105")
 					(unit 1)
 				)
@@
 		(dnp no)
 		(fields_autoplaced yes)
-		(property "Reference" "#PWR0107"
+		(property "Reference" "#PWR0108"
 			(at 72.39 71.12 0)
 			(effects
@@
 			(project "ECE145Mastermind"
 				(path "/8c64fe8a-5d6b-41bc-b3a3-9bda7b2e0f2c/9b9c62dc-9f79-4269-b727-e91a3c4aae61"
-					(reference "#PWR0107")
+					(reference "#PWR0108")
 					(unit 1)
 				)
@@
 		(dnp no)
 		(fields_autoplaced yes)
-		(property "Reference" "#PWR0106"
+		(property "Reference" "#PWR0107"
 			(at 72.39 43.18 0)
 			(effects
@@
 			(project "ECE145Mastermind"
 				(path "/8c64fe8a-5d6b-41bc-b3a3-9bda7b2e0f2c/9b9c62dc-9f79-4269-b727-e91a3c4aae61"
-					(reference "#PWR0106")
+					(reference "#PWR0107")
 					(unit 1)
 				)
@@
 		(dnp no)
 		(fields_autoplaced yes)
-		(property "Reference" "J8"
+		(property "Reference" "J12"
 			(at 55.245 57.15 0)
 			(effects
@@
 			(project "ECE145Mastermind"
 				(path "/8c64fe8a-5d6b-41bc-b3a3-9bda7b2e0f2c/9b9c62dc-9f79-4269-b727-e91a3c4aae61"
-					(reference "J8")
+					(reference "J12")
 					(unit 1)
 				)
@@
 		(dnp no)
 		(fields_autoplaced yes)
-		(property "Reference" "J6"
+		(property "Reference" "J10"
 			(at 42.545 57.15 0)
 			(effects
@@
 			(project "ECE145Mastermind"
 				(path "/8c64fe8a-5d6b-41bc-b3a3-9bda7b2e0f2c/9b9c62dc-9f79-4269-b727-e91a3c4aae61"
-					(reference "J6")
+					(reference "J10")
 					(unit 1)
 				)
@@
 		(dnp no)
 		(fields_autoplaced yes)
-		(property "Reference" "R28"
+		(property "Reference" "R29"
 			(at 49.53 55.8799 0)
 			(effects
@@
 			(project "ECE145Mastermind"
 				(path "/8c64fe8a-5d6b-41bc-b3a3-9bda7b2e0f2c/9b9c62dc-9f79-4269-b727-e91a3c4aae61"
-					(reference "R28")
+					(reference "R29")
 					(unit 1)
 				)
@@
 		(dnp no)
 		(fields_autoplaced yes)
-		(property "Reference" "#PWR0109"
+		(property "Reference" "#PWR0110"
 			(at 85.09 71.12 0)
 			(effects
@@
 			(project "ECE145Mastermind"
 				(path "/8c64fe8a-5d6b-41bc-b3a3-9bda7b2e0f2c/9b9c62dc-9f79-4269-b727-e91a3c4aae61"
-					(reference "#PWR0109")
+					(reference "#PWR0110")
 					(unit 1)
 				)
@@
 		(dnp no)
 		(fields_autoplaced yes)
-		(property "Reference" "#PWR0105"
+		(property "Reference" "#PWR0106"
 			(at 59.69 71.12 0)
 			(effects
@@
 			(project "ECE145Mastermind"
 				(path "/8c64fe8a-5d6b-41bc-b3a3-9bda7b2e0f2c/9b9c62dc-9f79-4269-b727-e91a3c4aae61"
-					(reference "#PWR0105")
-					(unit 1)
-				)
+					(reference "#PWR0106")
+					(unit 1)
+				)
