File: ECE145Mastermind.kicad_pcb (KiCad board)
At the start: 4 copper layers, 97 parts, among them J1 Conn_01x02_Socket, J10 Conn_01x01_Socket, J11 Conn_01x01_Socket, J12 Conn_01x01_Socket, J13 Conn_01x01_Socket, J14 Conn_01x01_Socket, J15 Conn_01x01_Socket, J16 Conn_01x01_Socket, J17 Conn_01x01_Socket, J2 Conn_01x01_Socket, J3 Conn_01x01_Socket, J4 Conn_01x01_Socket, J5 Conn_01x01_Socket, J6 Conn_01x01_Socket, J7 Conn_01x01_Socket, J8 Conn_01x01_Socket, J9 Conn_01x01_Socket, Q1 NMOS, SW1 SW_SPDT, SW2 SW_Push, U1 74LS08, U10 40106, U11 4053, U12 LM7805_TO220, U13 74LS194, U14 4053, U15 4051, U16 LM358, U17 LM324, U18 LM324, U19 74LS08, U2 74HCT00, U20 LM555xN, U21 74LS161, U22 74HCT00, U23 74HCT74, U24 74HCT00, U3 74LS73, U4 74LS194, U5 74LS148, U6 74LS73, U7 74LS194, U8 74LS139, U9 74HCT04

Commit message: For Sharvesh
Parts:
- added D9: LED, LED_SMD:LED_0805_2012Metric_Pad1.15x1.40mm_HandSolder, F.Cu at (223.0, 97.5)
- added R32: 1k, Resistor_SMD:R_0805_2012Metric_Pad1.20x1.40mm_HandSolder, F.Cu at (223.0, 100.5)
- moved U1 76.5 mm to (240.0, 59.0)
- moved U13 47.4 mm to (127.4, 52.5), turned to 90 degrees
- moved R12 24.7 mm to (118.5, 50.9), turned to 180 degrees
- moved U15 24.2 mm to (165.5, 33.4), turned to 180 degrees
- moved U2 23.1 mm to (132.0, 80.4), turned to 90 degrees
- moved U14 22.3 mm to (158.4, 44.5), turned to -90 degrees
- moved R20 21.8 mm to (116.5, 69.7)
- moved U16 21.7 mm to (168.5, 44.5), turned to -90 degrees
- moved R3 21.4 mm to (185.0, 47.5), turned to -90 degrees
- moved R21 18.8 mm to (117.3, 65.1), turned to -90 degrees
- moved R13 18.6 mm to (116.9, 46.8), turned to -90 degrees
- moved R11 17.8 mm to (102.8, 50.9)
- moved R19 17.2 mm to (104.8, 69.7), turned to 0 degrees
- moved R23 16.5 mm to (118.5, 56.5)
- moved R22 16.4 mm to (117.3, 60.6), turned to 90 degrees
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Connections:
- U1 pad 10: /Reset -> GND
- U1 pad 8: Net-(U7-Mr) -> unconnected-(U1-Pad8)
- U1 pad 9: PWR_ON_RST -> GND
- U19 pad 1: Net-(U18-Pad7) -> Net-(U18-Pad8)
- U19 pad 10: Net-(U17-Pad1) -> Net-(U17-Pad7)
- U19 pad 12: Net-(U17-Pad14) -> Net-(U17-Pad8)
- U19 pad 13: Net-(U17-Pad8) -> Net-(U17-Pad14)
- U19 pad 2: Net-(U18-Pad1) -> Net-(U18-Pad14)
- U19 pad 3: /Out1 -> /Out2
- U19 pad 4: Net-(U18-Pad14) -> Net-(U18-Pad1)
- U19 pad 5: Net-(U18-Pad8) -> Net-(U18-Pad7)
- U19 pad 6: /Out2 -> /Out1
- U19 pad 9: Net-(U17-Pad7) -> Net-(U17-Pad1)
- U7 pad 1: Net-(U7-Mr) -> Net-(U4-Mr)
Routing:
- net /J2: track 31.0 -> 0.00 mm
- net Net-(U11-Y1): track 0.00 -> 27.6 mm
- net /Out3: track 0.00 -> 23.9 mm
- net /Out4: track 0.00 -> 21.0 mm
- net /Out1: track 0.00 -> 19.6 mm
- net /Out2: track 0.00 -> 17.5 mm
- net Net-(U18-Pad14): track 0.00 -> 12.6 mm
- net Net-(U18-Pad1): track 0.00 -> 12.6 mm
- net Net-(U17-Pad8): track 0.00 -> 12.1 mm
- net Net-(U17-Pad7): track 0.00 -> 12.1 mm
- net /G4: track 0.00 -> 11.1 mm
- net /C2: track 0.00 -> 8.57 mm
- net /VB1: track 0.00 -> 8.02 mm
- net Net-(Q1-D): track 0.00 -> 7.94 mm
- net /G3: track 0.00 -> 7.85 mm
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
Commit message: routed
Parts:
- removed the D1 at (105.0, 165.5)
- added D9: LED, LED_SMD:LED_0603_1608Metric_Pad1.05x0.95mm_HandSolder, F.Cu at (114.7, 129.2)
- added R33: 1k, Capacitor_SMD:C_0805_2012Metric_Pad1.18x1.45mm_HandSolder, F.Cu at (103.0, 111.4)
- added R34: 1k, Capacitor_SMD:C_0805_2012Metric_Pad1.18x1.45mm_HandSolder, F.Cu at (113.7, 111.9)
- added R35: 1k, Capacitor_SMD:C_0805_2012Metric_Pad1.18x1.45mm_HandSolder, F.Cu at (94.9, 129.7)
- added R36: 1k, Capacitor_SMD:C_0805_2012Metric_Pad1.18x1.45mm_HandSolder, F.Cu at (119.8, 129.7)
- added R37: 2.2k, Capacitor_SMD:C_0805_2012Metric_Pad1.18x1.45mm_HandSolder, F.Cu at (99.5, 111.4)
- added R38: 2.2k, Capacitor_SMD:C_0805_2012Metric_Pad1.18x1.45mm_HandSolder, F.Cu at (110.2, 111.9)
- added R39: 2.2k, Capacitor_SMD:C_0805_2012Metric_Pad1.18x1.45mm_HandSolder, F.Cu at (94.9, 124.6)
- added R40: 2.2k, Capacitor_SMD:C_0805_2012Metric_Pad1.18x1.45mm_HandSolder, F.Cu at (119.8, 124.6)
- C12, C14: value 1u -> .1u
- D2, D3, D4, D5, D6, D7, D8: footprint LED_SMD:LED_0805_2012Metric_Pad1.15x1.40mm_HandSolder -> LED_SMD:LED_0603_1608Metric_Pad1.05x0.95mm_HandSolder
- R6: renamed from R5; value 200k -> 10k
- moved R5 119.3 mm to (168.7, 109.9), turned to 90 degrees
- moved U20 114.3 mm to (163.7, 106.9), turned to -90 degrees
- moved R6 113.0 mm to (170.7, 105.8), turned to 90 degrees
- moved J9 109.5 mm to (77.6, 132.8)
- moved C12 108.6 mm to (170.7, 101.8), turned to 90 degrees
- moved J7 108.2 mm to (68.1, 132.8)
- moved U22 107.2 mm to (167.9, 83.6), turned to 180 degrees
- moved J5 106.8 mm to (58.5, 132.8)
- moved J3 105.7 mm to (49.5, 132.6)
- moved C11 105.4 mm to (165.6, 113.5), turned to -90 degrees
- moved U23 104.9 mm to (159.3, 83.6)
- moved R8 103.8 mm to (174.2, 84.2), turned to 90 degrees
- moved R7 103.7 mm to (174.2, 79.9), turned to 90 degrees
- moved J8 101.1 mm to (77.6, 118.6)
- moved R28 101.1 mm to (77.6, 113.1)
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- renumbered D9 to D1, J6 to J10, J7 to J11, J8 to J12, J9 to J13, J10 to J3, J3 to J4, J4 to J5, J5 to J6, J11 to J7, J12 to J8, J13 to J9, R32 to R1, R9 to R10, R10 to R11, R11 to R12, R12 to R13, R13 to R14, R14 to R15, R15 to R16, R16 to R17, R17 to R18, R18 to R19, R1 to R2, R19 to R20, R20 to R21, R21 to R22, R22 to R23, R23 to R24, R24 to R25, R25 to R26, R26 to R27, R27 to R28, R28 to R29, R2 to R3, R29 to R30, R30 to R31, R31 to R32, R3 to R4, R4 to R5, R6 to R7, R7 to R8, R8 to R9
Connections:
- D2 pad 2: /Perfect LED/P2 -> Net-(D2-A)
- D3 pad 2: /Perfect LED/P3 -> Net-(D3-A)
- D4 pad 2: /Perfect LED/P4 -> Net-(D4-A)
- D5 pad 2: /Misplaced LED/M1 -> Net-(D5-A)
- D6 pad 2: /Misplaced LED/M2 -> Net-(D6-A)
- D7 pad 2: /Misplaced LED/M3 -> Net-(D7-A)
- D8 pad 2: /Misplaced LED/M4 -> Net-(D8-A)
- Q1 pad 1: Net-(Q1-D) -> Net-(Q1-G)
- Q1 pad 2: Net-(Q1-G) -> Net-(Q1-D)
- R10 pad 2: Net-(U18A--) -> Net-(U18D--)
- R11 pad 2: Net-(U18B--) -> Net-(U18C--)
- R12 pad 1: Net-(U18B--) -> Net-(U18C--)
- R13 pad 2: Net-(U18C--) -> Net-(U18A--)
- R14 pad 2: Net-(U18C--) -> Net-(U18A--)
- R15 pad 2: Net-(U18D--) -> Net-(U18B--)
- R16 pad 1: Net-(U18D--) -> Net-(U18B--)
- R9 pad 2: Net-(U18A--) -> Net-(U18D--)
- U10 pad 1: Net-(C14-Pad2) -> Net-(C1-Pad2)
- U10 pad 2: Net-(U10-Pad2) -> PWR_ON_RST
- U10 pad 3: Net-(C1-Pad2) -> Net-(C14-Pad2)
- U10 pad 4: PWR_ON_RST -> Net-(U10-Pad4)
- U18 pad 10: /VB2 -> /C1
- U18 pad 12: /C2 -> /VB1
- U18 pad 3: /VB1 -> /VB2
- U18 pad 5: /C1 -> /C2
- U19 pad 10: Net-(U17-Pad7) -> Net-(U17-Pad1)
- U19 pad 12: Net-(U17-Pad8) -> Net-(U17-Pad14)
- U19 pad 13: Net-(U17-Pad14) -> Net-(U17-Pad8)
- U19 pad 3: /Out2 -> /Out1
- U19 pad 4: Net-(U18-Pad1) -> Net-(U18-Pad7)
- U19 pad 5: Net-(U18-Pad7) -> Net-(U18-Pad1)
- U19 pad 6: /Out1 -> /Out2
- U19 pad 9: Net-(U17-Pad1) -> Net-(U17-Pad7)
- U2 pad 1: Net-(U3A-~{Q}) -> Net-(U3B-~{Q})
- U2 pad 10: /Out3 -> Net-(U6B-~{Q})
- U2 pad 11: Net-(U5-IO) -> Net-(U5-I3)
- U2 pad 12: Net-(U6B-~{Q}) -> Net-(U6A-~{Q})
- U2 pad 13: /Out4 -> /Out1
- U2 pad 2: /Out1 -> /Out4
- U2 pad 3: Net-(U5-I3) -> Net-(U5-IO)
- U2 pad 4: Net-(U3B-~{Q}) -> Net-(U3A-~{Q})
- U2 pad 5: /Out2 -> /Out3
- U2 pad 6: Net-(U5-I2) -> Net-(U5-I1)
- U2 pad 8: Net-(U5-I1) -> Net-(U5-I2)
- U2 pad 9: Net-(U6A-~{Q}) -> /Out2
- U22 pad 1: GND -> Net-(U10-Pad4)
- U22 pad 2: GND -> /Reset
- U22 pad 3: unconnected-(U22-Pad3) -> Net-(U22-Pad12)
- U22 pad 4: /Reset -> GND
- U22 pad 5: Net-(U22-Pad5) -> GND
- U22 pad 6: Net-(U23B-D) -> unconnected-(U22-Pad6)
- U22 pad 8: Net-(U22-Pad12) -> Net-(U23B-D)
- U22 pad 9: Net-(U10-Pad2) -> Net-(U22-Pad9)
- U24 pad 1: Net-(U24-Pad1) -> /P
- U24 pad 10: /DONE -> Net-(U24-Pad10)
- U24 pad 11: Net-(U23A-D) -> Net-(U22-Pad9)
- U24 pad 12: Net-(U24-Pad12) -> Net-(U24-Pad10)
- U24 pad 13: Net-(U24-Pad13) -> /P
- U24 pad 2: /P -> /DONE
- U24 pad 3: Net-(U22-Pad5) -> Net-(U24-Pad3)
- U24 pad 4: Net-(U24-Pad1) -> Net-(U24-Pad3)
- U24 pad 5: /M -> Net-(U24-Pad5)
- U24 pad 6: Net-(U24-Pad12) -> Net-(U23A-D)
- U24 pad 8: Net-(U24-Pad13) -> Net-(U24-Pad5)
- U24 pad 9: /P -> /M
- U3 pad 14: /J2 -> /J4
- U3 pad 7: /J1 -> /J3
- U4 pad 2: GND -> /P
- U4 pad 7: /P -> GND
- U6 pad 14: /J4 -> /J2
- U6 pad 7: /J3 -> /J1
- U7 pad 2: GND -> /M
- U7 pad 7: /M -> GND
- U9 pad 10: Net-(U24-Pad1) -> Net-(U24-Pad10)
Routing:
- net /CLK: track 0.00 -> 136.3 mm, vias 0 -> 3
- net /C1: track 4.49 -> 124.1 mm, vias 0 -> 2
- net /Reset: track 0.00 -> 119.5 mm, vias 0 -> 6
- net /C4: track 4.76 -> 109.8 mm, vias 0 -> 2
- net /C3: track 9.11 -> 110.7 mm
- net /G1: track 3.95 -> 102.4 mm
- net /M: track 0.00 -> 96.9 mm, vias 0 -> 2
- net /C2: track 8.57 -> 102.0 mm
- net /G2: track 4.10 -> 94.3 mm
- net /G3: track 7.85 -> 89.9 mm
- net /~{CLK}: track 0.00 -> 74.3 mm
- net /G4: track 11.1 -> 81.1 mm, vias 0 -> 2
- net Net-(U4-Mr): track 0.00 -> 67.5 mm, vias 0 -> 2
- net /P: track 0.00 -> 67.2 mm, vias 0 -> 6
- net /DONE: track 0.00 -> 65.0 mm, vias 0 -> 2
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Other:
- board outline added: 150.4 x 100.6 mm
- board text added: "Power On"

Commit message: Ground and Power Plane?
Parts:
- R33, R34, R35, R36, R37, R38, R39, R40: footprint Capacitor_SMD:C_0805_2012Metric_Pad1.18x1.45mm_HandSolder -> Resistor_SMD:R_0805_2012Metric_Pad1.20x1.40mm_HandSolder
- SW2: footprint Button_Switch_SMD:SW_SPST_Omron_B3FS-105xP -> Button_Switch_THT:SW_SPST_Omron_B3F-40xx
- moved C10 13.9 mm to (176.2, 103.8), turned to 0 degrees
- moved C4 8.49 mm to (134.5, 101.3), turned to 180 degrees
- moved SW2 2.19 mm to (132.2, 128.2)
- moved C6 1.18 mm to (165.0, 100.8)
- moved C5 1.07 mm to (152.8, 75.9), turned to 90 degrees
- moved R32 0.67 mm to (78.7, 57.1)
- moved C3 0.65 mm to (144.7, 115.5)
Connections:
- U19 pad 10: Net-(U17-Pad1) -> Net-(U17-Pad7)
- U19 pad 12: Net-(U17-Pad14) -> Net-(U17-Pad8)
- U19 pad 13: Net-(U17-Pad8) -> Net-(U17-Pad14)
- U19 pad 4: Net-(U18-Pad7) -> Net-(U18-Pad1)
- U19 pad 5: Net-(U18-Pad1) -> Net-(U18-Pad7)
- U19 pad 9: Net-(U17-Pad7) -> Net-(U17-Pad1)
Routing:
- net GND: track 0.00 -> 93.5 mm, vias 0 -> 67
- net Net-(C13-Pad2): track 9.79 -> 89.9 mm
- net Net-(U24-Pad10): track 4.37 -> 53.6 mm, vias 0 -> 2
- net +5V: track 0.00 -> 25.5 mm, vias 0 -> 48
- net /P: track 67.2 -> 61.0 mm
- net /M: track 96.9 -> 94.5 mm
- net /Reset: track 119.5 -> 121.4 mm
- net /DONE: track 65.0 -> 66.4 mm
- net Net-(U16B--): track 0.00 -> 1.27 mm
- net /G4: track 81.1 -> 81.8 mm
- added copper zone on In1.Cu, net +5V
- added copper zone on In2.Cu, net GND

Commit message: Finished?
Parts:
- added REF**: MountingHole_2.2mm_M2, MountingHole:MountingHole_2.2mm_M2, F.Cu at (190.6, 42.3)
- added REF**: MountingHole_2.2mm_M2, MountingHole:MountingHole_2.2mm_M2, F.Cu at (190.6, 134.3)
- added REF**: MountingHole_2.2mm_M2, MountingHole:MountingHole_2.2mm_M2, F.Cu at (48.6, 42.3)
- added REF**: MountingHole_2.2mm_M2, MountingHole:MountingHole_2.2mm_M2, F.Cu at (48.6, 134.3)
- added TP1: Out1, TestPoint:TestPoint_Pad_1.5x1.5mm, F.Cu at (123.3, 79.5)
- added TP2: Out2, TestPoint:TestPoint_Pad_1.5x1.5mm, F.Cu at (123.3, 83.8)
- added TP3: Out3, TestPoint:TestPoint_Pad_1.5x1.5mm, F.Cu at (123.3, 88.1)
- added TP4: Out4, TestPoint:TestPoint_Pad_1.5x1.5mm, F.Cu at (123.3, 92.4)
- added TP5: S0, TestPoint:TestPoint_Pad_1.5x1.5mm, F.Cu at (168.0, 97.0)
- added TP6: S1, TestPoint:TestPoint_Pad_1.5x1.5mm, F.Cu at (165.8, 91.9)
- added TP7: Clk, TestPoint:TestPoint_Pad_1.5x1.5mm, F.Cu at (171.6, 67.0)
- added TP8: M, TestPoint:TestPoint_Pad_1.5x1.5mm, F.Cu at (173.9, 62.7)
- added TP9: P, TestPoint:TestPoint_Pad_1.5x1.5mm, F.Cu at (173.9, 58.4)
- D2, D4, D6, D8: value LED -> White LED
- D3, D5, D7, D9: value LED -> Red LED
- J1: footprint Connector_PinSocket_1.27mm:PinSocket_1x02_P1.27mm_Vertical -> Connector_BarrelJack:BarrelJack_Horizontal
- J10, J11, J12, J13, J14, J15, J16, J17, J2, J3, J4, J5, J6, J7, J8, J9: footprint Connector_PinSocket_1.27mm:PinSocket_1x01_P1.27mm_Vertical -> Connector_PinSocket_2.54mm:PinSocket_1x01_P2.54mm_Vertical
- R10, R14, R18, R22: value 2.2k -> 10k
- R33, R35: value 1k -> 2.2k
- R38, R40: value 2.2k -> 1k
- moved SW2 69.8 mm to (100.0, 66.2)
- moved J9 16.4 mm to (86.8, 119.1)
- moved J7 16.1 mm to (76.6, 119.1)
- moved J5 15.8 mm to (66.4, 119.1)
- moved R36 15.5 mm to (105.7, 123.5), turned to 90 degrees
- moved J3 15.1 mm to (56.3, 119.1)
- moved R39 14.8 mm to (109.7, 123.6), turned to 90 degrees
- moved R33 13.6 mm to (114.7, 104.4)
- moved D5 13.6 mm to (103.9, 118.5), turned to -90 degrees
- moved R28 13.6 mm to (86.8, 103.1)
- moved D8 13.5 mm to (111.4, 118.5), turned to -90 degrees
- moved J8 13.3 mm to (86.8, 109.0)
- moved D2 13.1 mm to (112.9, 109.5)
- moved R27 13.0 mm to (76.4, 103.1)
- moved J6 12.9 mm to (76.6, 109.0)
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- renumbered C2 to C1, C3 to C2, C4 to C3, C5 to C4, C6 to C5, C7 to C6, C1 to C7, U11 to U10, U13 to U11, U14 to U12, U15 to U13, U10 to U14, U16 to U15, U12 to U16, U6 to U3, U3 to U6
Connections:
- net /Misplaced LED/M1 renamed /M1
- net /Perfect LED/P2 renamed /P2
- R33 pad 1: /Perfect LED/P1 -> /M2
- R35 pad 1: /Perfect LED/P3 -> /M3
- R36 pad 1: /Perfect LED/P4 -> /P3
- R38 pad 1: /Misplaced LED/M2 -> /P1
- R39 pad 1: /Misplaced LED/M3 -> /M4
- R40 pad 1: /Misplaced LED/M4 -> /P4
- U4 pad 12: /Perfect LED/P4 -> /P4
- U4 pad 13: /Perfect LED/P3 -> /P3
- U4 pad 15: /Perfect LED/P1 -> /P1
- U7 pad 12: /Misplaced LED/M4 -> /M4
- U7 pad 13: /Misplaced LED/M3 -> /M3
- U7 pad 14: /Misplaced LED/M2 -> /M2
Routing:
- net /Perfect LED/P3: track 50.1 -> 0.00 mm
- net /Misplaced LED/M3: track 37.9 -> 0.00 mm, vias 2 -> 0
- net /P1: track 0.00 -> 36.6 mm
- net /P3: track 0.00 -> 34.5 mm
- net /M3: track 0.00 -> 33.7 mm
- net /Perfect LED/P1: track 32.6 -> 0.00 mm
- net /M2: track 0.00 -> 29.8 mm, vias 0 -> 2
- net /Perfect LED/P4: track 29.0 -> 0.00 mm
- net /Misplaced LED/M2: track 27.1 -> 0.00 mm, vias 2 -> 0
- net /P4: track 0.00 -> 25.5 mm
- net /M4: track 0.00 -> 23.2 mm
- net Net-(C13-Pad2): track 89.9 -> 112.5 mm, vias 0 -> 1
- net /C4: track 110.2 -> 91.0 mm
- net /M: track 94.5 -> 113.4 mm, vias 2 -> 4
- net /C3: track 110.7 -> 92.3 mm
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Other:
- board size 150.4 x 100.6 mm -> 150 x 100 mm

Commit message: Final touches
Parts:
- added REF**: MountingHole_2.2mm_M2, MountingHole:MountingHole_2.2mm_M2, F.Cu at (94.1, 81.9)
- added REF**: MountingHole_2.2mm_M2, MountingHole:MountingHole_2.2mm_M2, F.Cu at (48.6, 81.9)
- REF** (x4): value MountingHole_2.2mm_M2 -> MountingHole_3.2mm_M3; footprint MountingHole:MountingHole_2.2mm_M2 -> MountingHole:MountingHole_3.2mm_M3
- TP5: renamed from TP8; value M -> S0
- TP6: renamed from TP9; value P -> S1
- TP7: renamed from TP5; value S0 -> Clk
- TP8: renamed from TP7; value Clk -> M
- TP9: renamed from TP6; value S1 -> P
- moved J2 2.00 mm to (56.3, 111.0)
- moved J3 2.00 mm to (56.3, 121.1)
- moved J4 2.00 mm to (66.4, 111.0)
- moved J5 2.00 mm to (66.4, 121.1)
- moved J6 2.00 mm to (76.6, 111.0)
- moved J7 2.00 mm to (76.6, 121.1)
- moved J8 2.00 mm to (86.8, 111.0)
- moved J9 2.00 mm to (86.8, 121.1)
- moved R25 2.00 mm to (56.0, 105.1)
- moved R26 2.00 mm to (66.4, 105.1)
- moved R27 2.00 mm to (76.4, 105.1)
- moved R28 2.00 mm to (86.8, 105.1)
Connections:
- TP5 pad 1: /M -> /S0
- TP6 pad 1: /P -> /S1
- TP7 pad 1: /S0 -> /CLK
- TP8 pad 1: /CLK -> /M
- TP9 pad 1: /S1 -> /P
Routing:
- net Net-(C13-Pad2): track 112.5 -> 125.0 mm
- net /C4: track 91.0 -> 98.0 mm
- net /C2: track 84.0 -> 91.1 mm
- net /C3: track 92.3 -> 99.3 mm
- net /C1: track 107.8 -> 114.8 mm
- net GND: track 93.5 -> 99.5 mm, vias 73 -> 63
Other:
- board text added: "ECE 145 Spring 2026"

Commit message: trying things out
Parts:
- moved C1 2.26 mm to (153.3, 58.9)
Connections:
- U1 pad 11: unconnected-(U1-Pad11) -> Net-(U4-S0)
- U1 pad 12: GND -> Net-(U5-EO)
- U1 pad 13: GND -> /FSM/~{Wait}
- U22 pad 4: GND -> Net-(U23A-~{Q})
- U22 pad 5: GND -> Net-(U23B-~{Q})
- U22 pad 6: unconnected-(U22-Pad6) -> /FSM/~{Wait}
- U23 pad 6: unconnected-(U23A-~{Q}-Pad6) -> Net-(U23A-~{Q})
- U5 pad 15: Net-(U4-S0) -> Net-(U5-EO)
Routing:
- net Net-(U4-S0): track 45.2 -> 104.8 mm, vias 2 -> 4
- net Net-(U5-EO): track 0.00 -> 58.2 mm, vias 0 -> 2
- net /FSM/~{Wait}: track 0.00 -> 31.9 mm, vias 0 -> 2
- net Net-(U23A-~{Q}): track 0.00 -> 14.6 mm
- net Net-(U23B-~{Q}): track 4.21 -> 15.8 mm
- net GND: track 99.5 -> 90.7 mm, vias 63 -> 61
- net Net-(U4-Mr): track 67.5 -> 75.8 mm
- net /DONE: track 66.4 -> 73.9 mm
- net Net-(Q1-G): track 46.0 -> 52.8 mm
- net /Reset: track 122.6 -> 129.3 mm
- net /M: track 113.4 -> 116.7 mm
- net /CLK: track 147.2 -> 148.4 mm
