File: ECE145Mastermind.kicad_sch (KiCad schematic)
At the start: 44 parts, among them J1 Conn_01x02_Socket, Q1 NMOS, SW1 SW_SPDT, U1 74LS08, U10 40106, U11 4053, U12 LM7805_TO220, U13 74LS194, U14 4053, U15 4051, U16 LM358, U17 LM324, U18 LM324, U19 74LS08, U2 74HCT00, U20 LM555xN, U21 74LS161, U22 74HCT00, U3 74LS73, U4 74LS194, U5 74LS148, U6 74LS73, U7 74LS194, U8 74LS139, U9 74HCT04

Commit message: Finished?
Parts:
- added TP1: Out1, TestPoint:TestPoint_Pad_1.5x1.5mm, symbol Connector:TestPoint_Small
- added TP2: Out2, TestPoint:TestPoint_Pad_1.5x1.5mm, symbol Connector:TestPoint_Small
- added TP3: Out3, TestPoint:TestPoint_Pad_1.5x1.5mm, symbol Connector:TestPoint_Small
- added TP4: Out4, TestPoint:TestPoint_Pad_1.5x1.5mm, symbol Connector:TestPoint_Small
- added TP5: Clk, TestPoint:TestPoint_Pad_1.5x1.5mm, symbol Connector:TestPoint_Small
- added TP8: S0, TestPoint:TestPoint_Pad_1.5x1.5mm, symbol Connector:TestPoint_Small
- added TP9: S1, TestPoint:TestPoint_Pad_1.5x1.5mm, symbol Connector:TestPoint_Small
- J1: footprint Connector_PinSocket_1.27mm:PinSocket_1x02_P1.27mm_Vertical -> Connector_BarrelJack:BarrelJack_Horizontal; symbol Connector:Conn_01x02_Socket -> Connector:Barrel_Jack
- renumbered C2 to C1, C3 to C2, C4 to C3, C5 to C4, C6 to C5, C7 to C6, C1 to C7, U11 to U10, U13 to U11, U14 to U12, U15 to U13, U10 to U14, U16 to U15, U12 to U16, U6 to U3, U3 to U6
Connections:
- net CLK: now also TP5.1
- net Out1: now also TP1.1
- net Out2: now also TP2.1
- net Out3: now also TP3.1
- net Out4: now also TP4.1
- net S0: now also TP8.1
- net S1: now also TP9.1
- net Misplaced LED/M1 renamed M1
- net Misplaced LED/M2 renamed M2
- net Misplaced LED/M3 renamed M3
- net Misplaced LED/M4 renamed M4
- net Perfect LED/P1 renamed P1
- net Perfect LED/P2 renamed P2
- net Perfect LED/P3 renamed P3
- net Perfect LED/P4 renamed P4
Other:
- removed sheet Guess
- removed sheet Misplaced LED
- removed sheet Perfect LED
- added sheet Code1 (Code.kicad_sch)
- added sheet LED (bicolor LED.kicad_sch)
- added sheet LED1 (bicolor LED.kicad_sch)
- added sheet LED2 (bicolor LED.kicad_sch)
- added sheet LED3 (bicolor LED.kicad_sch)
- moved on the sheet: C7, D1, R1, R2, SW1, U14A, U16, U7

Commit message: Final touches
Parts:
- renumbered TP8 to TP5, TP9 to TP6, TP5 to TP7
Changed lines of the file:
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@@
 		(dnp no)
 		(fields_autoplaced yes)
-		(property "Reference" "TP8"
+		(property "Reference" "TP5"
 			(at 288.29 39.37 90)
 			(show_name no)
@@
 			(project "ECE145Mastermind"
 				(path "/8c64fe8a-5d6b-41bc-b3a3-9bda7b2e0f2c"
-					(reference "TP8")
+					(reference "TP5")
 					(unit 1)
 				)
@@
 		(in_pos_files yes)
 		(dnp no)
-		(property "Reference" "TP5"
+		(property "Reference" "TP7"
 			(at 318.77 82.5499 0)
 			(show_name no)
@@
 			(project "ECE145Mastermind"
 				(path "/8c64fe8a-5d6b-41bc-b3a3-9bda7b2e0f2c"
-					(reference "TP5")
+					(reference "TP7")
 					(unit 1)
 				)
@@
 		(in_pos_files yes)
 		(dnp no)
-		(property "Reference" "TP9"
+		(property "Reference" "TP6"
 			(at 307.34 36.83 90)
 			(show_name no)
@@
 			(project "ECE145Mastermind"
 				(path "/8c64fe8a-5d6b-41bc-b3a3-9bda7b2e0f2c"
-					(reference "TP9")
-					(unit 1)
-				)
+					(reference "TP6")
+					(unit 1)
+				)

Commit message: trying things out
Parts:
- removed U22: 74HCT00, Package_SO:SOIC-14_3.9x8.7mm_P1.27mm, symbol 74xx:74HCT00
Connections:
- net GND: no longer U1.12, U1.13
- net at U1.11: now also U4.9 (S0), U7.9 (S0)
- new net: U1.12, U5.15 (EO)
- new net FSM/~{Wait}: U1.13
- no-connect marks 32 -> 30
Other:
- sheet FSM ports: added ~{Wait}; removed none
- moved on the sheet: TP7

Commit message: made things nice
Parts:
- removed unit 4 of U1
- removed unit 6 of U9
- added U22: 74HCT00, Package_SO:SOIC-14_3.9x8.7mm_P1.27mm, symbol 74xx:74HCT00
- added unit 6 of U3
- renumbered TP7 to TP5, TP5 to TP6, TP6 to TP7, U9 to U3, U3 to U4, U4 to U5, U5 to U6, U6 to U7, U7 to U8, U8 to U9
Connections:
- net CLK: now also U22.4, U22.5
- net GND: no longer U6.5 (EI)
- net ~{CLK}: now also U22.6
- net at U6.14 (GS), U9.1 (E): now also U3.13
- net at U5.9 (S0), U8.9 (S0): now also U3.12
- new net WAIT: U6.5 (EI)
- no-connect marks 30 -> 31
Other:
- sheet FSM ports: added WAIT; removed ~{Wait}
