File: FSM.kicad_sch (KiCad schematic)
At the start: 12 parts, among them SW2 SW_Push, U14 40106, U22 74HCT00, U23 74HCT74, U24 74HCT00, U9 74HCT04

Commit message: trying things out
Parts:
- added unit 2 of U22
Connections:
- net at U22.13, U23.8 (~{Q}): now also U22.5
- net at U23.6 (~{Q}): now also U22.4
- new net ~{Wait}: U22.6
- no-connect marks 1 -> 0
Changed lines of the file:
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@@
 	)
 	(junction
+		(at 92.71 35.56)
+		(diameter 0)
+		(color 0 0 0 0)
+	)
+	(junction
 		(at 118.11 38.1)
 		(diameter 0)
@@
 		(color 0 0 0 0)
 	)
-	(no_connect
-		(at 90.17 62.23)
-	)
 	(wire
 		(pts
@@
 	(wire
 		(pts
+			(xy 90.17 90.17) (xy 85.09 90.17)
+		)
+		(stroke
+			(width 0)
+			(type default)
+		)
+	)
+	(wire
+		(pts
 			(xy 118.11 19.05) (xy 118.11 38.1)
 		)
@@
 	(wire
 		(pts
+			(xy 85.09 95.25) (xy 92.71 95.25)
+		)
+		(stroke
+			(width 0)
+			(type default)
+		)
+	)
+	(wire
+		(pts
 			(xy 90.17 57.15) (xy 93.98 57.15)
 		)
@@
 	(wire
 		(pts
+			(xy 92.71 35.56) (xy 102.87 35.56)
+		)
+		(stroke
+			(width 0)
+			(type default)
+		)
+	)
+	(wire
+		(pts
 			(xy 96.52 92.71) (xy 96.52 93.98)
 		)
@@
 	(wire
 		(pts
+			(xy 90.17 62.23) (xy 90.17 90.17)
+		)
+		(stroke
+			(width 0)
+			(type default)
+		)
+	)
+	(wire
+		(pts
 			(xy 40.64 30.48) (xy 44.45 30.48)
 		)
@@
 	(wire
 		(pts
-			(xy 90.17 35.56) (xy 102.87 35.56)
+			(xy 90.17 35.56) (xy 92.71 35.56)
 		)
 		(stroke
@@
 	(wire
 		(pts
+			(xy 92.71 95.25) (xy 92.71 35.56)
+		)
+		(stroke
+			(width 0)
+			(type default)
+		)
+	)
+	(wire
+		(pts
 			(xy 43.18 21.59) (xy 93.98 21.59)
 		)
@@
 		)
 	)
+	(hierarchical_label "~{Wait}"
+		(shape output)
+		(at 69.85 92.71 180)
+		(effects
+			(font
+				(size 1.27 1.27)
+			)
+			(justify right)
+		)
+	)
 	(hierarchical_label "DONE"
 		(shape input)
@@
 				)
 			)
+		)
+	)
+	(symbol
+		(lib_id "74xx:74HCT00")
+		(at 77.47 92.71 0)
+		(mirror y)
+		(unit 2)
+		(body_style 1)
+		(exclude_from_sim no)
+		(in_bom yes)
+		(on_board yes)
+		(in_pos_files yes)
+		(dnp no)
+		(fields_autoplaced yes)
+		(property "Reference" "U22"
+			(at 77.4783 83.82 0)
+			(show_name no)
+			(do_not_autoplace no)
+			(effects
+				(font
+					(size 1.27 1.27)
+				)
+			)
+		)
+		(property "Value" "74HCT00"
+			(at 77.4783 86.36 0)
+			(show_name no)
+			(do_not_autoplace no)
+			(effects
+				(font
+					(size 1.27 1.27)
+				)
+			)
+		)
+		(property "Footprint" "Package_SO:SOIC-14_3.9x8.7mm_P1.27mm"
+			(at 77.47 92.71 0)
+			(hide yes)
+			(show_name no)
+			(do_not_autoplace no)
+			(effects
+				(font
+					(size 1.27 1.27)
+				)
+			)
+		)
+		(property "Datasheet" "http://www.ti.com/lit/gpn/sn74hct00"
+			(at 77.47 92.71 0)
+			(hide yes)
+			(show_name no)
+			(do_not_autoplace no)
+			(effects
+				(font
+					(size 1.27 1.27)
+				)
+			)
+		)
+		(property "Description" "quad 2-input NAND gate"
+			(at 77.47 92.71 0)
+			(hide yes)
+			(show_name no)
+			(do_not_autoplace no)
+			(effects
+				(font
+					(size 1.27 1.27)
+				)
+			)
+		)
+		(pin "13"
+		)
+		(pin "12"
+		)
+		(pin "8"
+		)
+		(pin "10"
+		)
+		(pin "9"
+		)
+		(pin "2"
+		)
+		(pin "1"
+		)
+		(pin "4"
+		)
+		(pin "5"
+		)
+		(pin "3"
+		)
+		(pin "6"
+		)
+		(pin "11"
+		)
+		(pin "14"
+		)
+		(pin "7"
+		)
+		(instances
+			(project "ECE145Mastermind"
+				(path "/8c64fe8a-5d6b-41bc-b3a3-9bda7b2e0f2c/c249946c-91e3-42cd-8f8a-d6059405d3e8"
+					(reference "U22")
+					(unit 2)
+				)
+			)

Commit message: made things nice
Parts:
- removed unit 2 of U22
- added U1: 74LS08, Package_SO:SOIC-14_3.9x8.7mm_P1.27mm, symbol 74xx:74LS08
- renumbered U9 to U3
Connections:
- net at U23.6 (~{Q}): now also U1.13
- net at U22.13, U23.8 (~{Q}): now also U1.12
- new net WAIT: U1.11
Changed lines of the file:
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@@
 		)
 	)
-	(hierarchical_label "~{Wait}"
+	(hierarchical_label "WAIT"
 		(shape output)
 		(at 69.85 92.71 180)
@@
 		(dnp no)
 		(fields_autoplaced yes)
-		(property "Reference" "#PWR076"
+		(property "Reference" "#PWR075"
 			(at 20.32 95.25 0)
 			(hide yes)
@@
 			(project "ECE145Mastermind"
 				(path "/8c64fe8a-5d6b-41bc-b3a3-9bda7b2e0f2c/c249946c-91e3-42cd-8f8a-d6059405d3e8"
-					(reference "#PWR076")
+					(reference "#PWR075")
 					(unit 1)
 				)
@@
 		(dnp no)
 		(fields_autoplaced yes)
-		(property "Reference" "#PWR081"
+		(property "Reference" "#PWR080"
 			(at 63.5 132.08 0)
 			(hide yes)
@@
 			(project "ECE145Mastermind"
 				(path "/8c64fe8a-5d6b-41bc-b3a3-9bda7b2e0f2c/c249946c-91e3-42cd-8f8a-d6059405d3e8"
-					(reference "#PWR081")
+					(reference "#PWR080")
 					(unit 1)
 				)
@@
 		(dnp no)
 		(fields_autoplaced yes)
-		(property "Reference" "#PWR085"
+		(property "Reference" "#PWR084"
 			(at 116.84 76.2 0)
 			(hide yes)
@@
 			(project "ECE145Mastermind"
 				(path "/8c64fe8a-5d6b-41bc-b3a3-9bda7b2e0f2c/c249946c-91e3-42cd-8f8a-d6059405d3e8"
-					(reference "#PWR085")
+					(reference "#PWR084")
 					(unit 1)
 				)
@@
 		(dnp no)
 		(fields_autoplaced yes)
-		(property "Reference" "#PWR083"
+		(property "Reference" "#PWR082"
 			(at 82.55 55.88 0)
 			(hide yes)
@@
 			(project "ECE145Mastermind"
 				(path "/8c64fe8a-5d6b-41bc-b3a3-9bda7b2e0f2c/c249946c-91e3-42cd-8f8a-d6059405d3e8"
-					(reference "#PWR083")
+					(reference "#PWR082")
 					(unit 1)
 				)
@@
 		(dnp no)
 		(fields_autoplaced yes)
-		(property "Reference" "#PWR079"
+		(property "Reference" "#PWR078"
 			(at 41.91 132.08 0)
 			(hide yes)
@@
 			(project "ECE145Mastermind"
 				(path "/8c64fe8a-5d6b-41bc-b3a3-9bda7b2e0f2c/c249946c-91e3-42cd-8f8a-d6059405d3e8"
-					(reference "#PWR079")
+					(reference "#PWR078")
 					(unit 1)
-				)
-			)
-		)
-	)
-	(symbol
-		(lib_id "74xx:74HCT00")
-		(at 77.47 92.71 0)
-		(mirror y)
-		(unit 2)
-		(body_style 1)
-		(exclude_from_sim no)
-		(in_bom yes)
-		(on_board yes)
-		(in_pos_files yes)
-		(dnp no)
-		(fields_autoplaced yes)
-		(property "Reference" "U22"
-			(at 77.4783 83.82 0)
-			(show_name no)
-			(do_not_autoplace no)
-			(effects
-				(font
-					(size 1.27 1.27)
-				)
-			)
-		)
-		(property "Value" "74HCT00"
-			(at 77.4783 86.36 0)
-			(show_name no)
-			(do_not_autoplace no)
-			(effects
-				(font
-					(size 1.27 1.27)
-				)
-			)
-		)
-		(property "Footprint" "Package_SO:SOIC-14_3.9x8.7mm_P1.27mm"
-			(at 77.47 92.71 0)
-			(hide yes)
-			(show_name no)
-			(do_not_autoplace no)
-			(effects
-				(font
-					(size 1.27 1.27)
-				)
-			)
-		)
-		(property "Datasheet" "http://www.ti.com/lit/gpn/sn74hct00"
-			(at 77.47 92.71 0)
-			(hide yes)
-			(show_name no)
-			(do_not_autoplace no)
-			(effects
-				(font
-					(size 1.27 1.27)
-				)
-			)
-		)
-		(property "Description" "quad 2-input NAND gate"
-			(at 77.47 92.71 0)
-			(hide yes)
-			(show_name no)
-			(do_not_autoplace no)
-			(effects
-				(font
-					(size 1.27 1.27)
-				)
-			)
-		)
-		(pin "13"
-		)
-		(pin "12"
-		)
-		(pin "8"
-		)
-		(pin "10"
-		)
-		(pin "9"
-		)
-		(pin "2"
-		)
-		(pin "1"
-		)
-		(pin "4"
-		)
-		(pin "5"
-		)
-		(pin "3"
-		)
-		(pin "6"
-		)
-		(pin "11"
-		)
-		(pin "14"
-		)
-		(pin "7"
-		)
-		(instances
-			(project "ECE145Mastermind"
-				(path "/8c64fe8a-5d6b-41bc-b3a3-9bda7b2e0f2c/c249946c-91e3-42cd-8f8a-d6059405d3e8"
-					(reference "U22")
-					(unit 2)
 				)
 			)
@@
 		(dnp no)
 		(fields_autoplaced yes)
-		(property "Reference" "#PWR077"
+		(property "Reference" "#PWR076"
 			(at 20.32 129.54 0)
 			(hide yes)
@@
 			(project "ECE145Mastermind"
 				(path "/8c64fe8a-5d6b-41bc-b3a3-9bda7b2e0f2c/c249946c-91e3-42cd-8f8a-d6059405d3e8"
-					(reference "#PWR077")
+					(reference "#PWR076")
 					(unit 1)
 				)
@@
 		(dnp no)
 		(fields_autoplaced yes)
-		(property "Reference" "U9"
+		(property "Reference" "U3"
 			(at 33.02 21.59 0)
 			(show_name no)
@@
 			(project "ECE145Mastermind"
 				(path "/8c64fe8a-5d6b-41bc-b3a3-9bda7b2e0f2c/c249946c-91e3-42cd-8f8a-d6059405d3e8"
-					(reference "U9")
+					(reference "U3")
 					(unit 5)
 				)
@@
 		(dnp no)
 		(fields_autoplaced yes)
-		(property "Reference" "#PWR084"
+		(property "Reference" "#PWR083"
 			(at 102.87 101.6 0)
 			(hide yes)
@@
 			(project "ECE145Mastermind"
 				(path "/8c64fe8a-5d6b-41bc-b3a3-9bda7b2e0f2c/c249946c-91e3-42cd-8f8a-d6059405d3e8"
-					(reference "#PWR084")
+					(reference "#PWR083")
 					(unit 1)
 				)
@@
 		(dnp no)
 		(fields_autoplaced yes)
-		(property "Reference" "#PWR080"
+		(property "Reference" "#PWR079"
 			(at 63.5 104.14 0)
 			(hide yes)
@@
 			(project "ECE145Mastermind"
 				(path "/8c64fe8a-5d6b-41bc-b3a3-9bda7b2e0f2c/c249946c-91e3-42cd-8f8a-d6059405d3e8"
-					(reference "#PWR080")
+					(reference "#PWR079")
 					(unit 1)
+				)
+			)
+		)
+	)
+	(symbol
+		(lib_id "74xx:74LS08")
+		(at 77.47 92.71 180)
+		(unit 4)
+		(body_style 1)
+		(exclude_from_sim no)
+		(in_bom yes)
+		(on_board yes)
+		(in_pos_files yes)
+		(dnp no)
+		(fields_autoplaced yes)
+		(property "Reference" "U1"
+			(at 77.4783 83.82 0)
+			(show_name no)
+			(do_not_autoplace no)
+			(effects
+				(font
+					(size 1.27 1.27)
+				)
+			)
+		)
+		(property "Value" "74LS08"
+			(at 77.4783 86.36 0)
+			(show_name no)
+			(do_not_autoplace no)
+			(effects
+				(font
+					(size 1.27 1.27)
+				)
+			)
+		)
+		(property "Footprint" "Package_SO:SOIC-14_3.9x8.7mm_P1.27mm"
+			(at 77.47 92.71 0)
+			(hide yes)
+			(show_name no)
+			(do_not_autoplace no)
+			(effects
+				(font
+					(size 1.27 1.27)
+				)
+			)
+		)
+		(property "Datasheet" "http://www.ti.com/lit/gpn/sn74LS08"
+			(at 77.47 92.71 0)
+			(hide yes)
+			(show_name no)
+			(do_not_autoplace no)
+			(effects
+				(font
+					(size 1.27 1.27)
+				)
+			)
+		)
+		(property "Description" "Quad And2"
+			(at 77.47 92.71 0)
+			(hide yes)
+			(show_name no)
+			(do_not_autoplace no)
+			(effects
+				(font
+					(size 1.27 1.27)
+				)
+			)
+		)
+		(pin "9"
+		)
+		(pin "12"
+		)
+		(pin "10"
+		)
+		(pin "13"
+		)
+		(pin "8"
+		)
+		(pin "11"
+		)
+		(pin "1"
+		)
+		(pin "2"
+		)
+		(pin "3"
+		)
+		(pin "5"
+		)
+		(pin "4"
+		)
+		(pin "6"
+		)
+		(pin "14"
+		)
+		(pin "7"
+		)
+		(instances
+			(project "ECE145Mastermind"
+				(path "/8c64fe8a-5d6b-41bc-b3a3-9bda7b2e0f2c/c249946c-91e3-42cd-8f8a-d6059405d3e8"
+					(reference "U1")
+					(unit 4)
 				)
 			)
@@
 		(dnp no)
 		(fields_autoplaced yes)
-		(property "Reference" "#PWR078"
+		(property "Reference" "#PWR077"
 			(at 41.91 104.14 0)
 			(hide yes)
@@
 			(project "ECE145Mastermind"
 				(path "/8c64fe8a-5d6b-41bc-b3a3-9bda7b2e0f2c/c249946c-91e3-42cd-8f8a-d6059405d3e8"
-					(reference "#PWR078")
+					(reference "#PWR077")
 					(unit 1)
 				)
@@
 		(dnp no)
 		(fields_autoplaced yes)
-		(property "Reference" "#PWR086"
+		(property "Reference" "#PWR085"
 			(at 116.84 83.82 0)
 			(hide yes)
@@
 			(project "ECE145Mastermind"
 				(path "/8c64fe8a-5d6b-41bc-b3a3-9bda7b2e0f2c/c249946c-91e3-42cd-8f8a-d6059405d3e8"
-					(reference "#PWR086")
+					(reference "#PWR085")
 					(unit 1)
 				)
@@
 		(dnp no)
 		(fields_autoplaced yes)
-		(property "Reference" "#PWR082"
+		(property "Reference" "#PWR081"
 			(at 82.55 29.21 0)
 			(hide yes)
@@
 			(project "ECE145Mastermind"
 				(path "/8c64fe8a-5d6b-41bc-b3a3-9bda7b2e0f2c/c249946c-91e3-42cd-8f8a-d6059405d3e8"
-					(reference "#PWR082")
+					(reference "#PWR081")
 					(unit 1)
 				)
