File: Design Blocks/Mastermind.kicad_blocks/Code.kicad_block/Code.kicad_sch (KiCad schematic)
At the start: 12 parts, among them J10 Conn_01x01_Socket, J11 Conn_01x01_Socket, J12 Conn_01x01_Socket, J13 Conn_01x01_Socket, J14 Conn_01x01_Socket, J15 Conn_01x01_Socket, J16 Conn_01x01_Socket, J17 Conn_01x01_Socket

Commit message: Finished?
Parts:
- removed J10, J11, J12, J13, J14, J15, J16, J17: Conn_01x01_Socket, Connector_PinSocket_1.27mm:PinSocket_1x01_P1.27mm_Vertical, symbol Connector:Conn_01x01_Socket
- removed R29, R30, R31, R32: 10k, Resistor_SMD:R_0805_2012Metric_Pad1.20x1.40mm_HandSolder, symbol Device:R
- added J2, J3, J4, J5, J6, J7, J8, J9: Conn_01x01_Socket, Connector_PinSocket_2.54mm:PinSocket_1x01_P2.54mm_Vertical, symbol Connector:Conn_01x01_Socket
- added R25, R26, R27, R28: 10k, Resistor_SMD:R_0805_2012Metric_Pad1.20x1.40mm_HandSolder, symbol Device:R
Connections:
- net +5V: now also R25.1, R26.1, R27.1, R28.1
- net GND: now also J3.1 (Pin_1), J5.1 (Pin_1), J7.1 (Pin_1), J9.1 (Pin_1)
- new net C1: J2.1 (Pin_1), R25.2
- new net C2: J4.1 (Pin_1), R26.2
- new net C3: J6.1 (Pin_1), R27.2
- new net C4: J8.1 (Pin_1), R28.2
Other:
- title: Guess Input Voltage Dividers -> Code INput Voltage Dividers
